Commit message: Simulation test for not collision but still only wheels collide

File: multi_turtlebot_sim/urdf/gazebo_specific.urdf.xacro (robot description, xacro)
@@ -1,5 +1,54 @@
 <?xml version="1.0"?>
 <robot xmlns:xacro="http://ros.org/wiki/xacro" name="noah_wheel">
-	<xacro:macro name="gazebo_specific" params="frame_prefix topic_prefix">
+	<xacro:macro name="gazebo_specific" params="frame_prefix topic_prefix collision_bitmap">
+    <gazebo>
+      <static>false</static>
+      <self_collide>false</self_collide>
+    </gazebo>
+    <gazebo reference="base_link">
+      <material>Gazebo/Black</material>
+      <collision>
+        <surface>
+          <contact>
+            <collide_without_contact>true</collide_without_contact>
+            <collide_without_contact_bitmask>0x0F</collide_without_contact_bitmask>
+          </contact>
+        </surface>
+      </collision>
+    </gazebo>
+    <gazebo reference="wheel_left_link">
+      <material>Gazebo/DarkGrey</material>
+      <collision>
+        <surface>
+          <contact>
+            <collide_without_contact>false</collide_without_contact>
+            <collide_bitmask>0x0F</collide_bitmask>
+          </contact>
+          <friction>
+            <ode>
+              <mu>1.0</mu>
+              <mu2>1.0</mu2>
+            </ode>
+          </friction>
+        </surface>
+      </collision>
+    </gazebo>
+    <gazebo reference="wheel_right_link">
+      <material>Gazebo/DarkGrey</material>
+      <collision>
+        <surface>
+          <contact>
+            <collide_without_contact>false</collide_without_contact>
+            <collide_bitmask>0x0F</collide_bitmask>
+          </contact>
+          <friction>
+            <ode>
+              <mu>1.0</mu>
+              <mu2>1.0</mu2>
+            </ode>
+          </friction>
+        </surface>
+      </collision>
+    </gazebo>
     <gazebo>
       <plugin name="turtlebot3_diff_drive" filename="libgazebo_ros_diff_drive.so">

File: multi_turtlebot_sim/urdf/turtlebot3_waffle.urdf.xacro (robot description, xacro)
@@ -12,4 +12,6 @@
   <xacro:arg name="topic_prefix" default=""/>
   <xacro:property name="topic_prefix" value="$(arg topic_prefix)"/>
+  <xacro:arg name="collision_bitmap" default="0x01"/>
+  <xacro:property name="collision_bitmap" value="$(arg collision_bitmap)"/>
   <!-- "package://" isn't working with gazebo_ros ROS2(package is replaced by model) so it worked as a workaround to find the meshes -->
   <xacro:property name="meshes_folder" value="$(find multi_turtlebot_sim)/meshes"/>
@@ -59,11 +61,11 @@
       <material name="light_black"/>
     </visual>
-    <!-- <collision>
+    <collision>
       <origin xyz="-0.064 0 0.047" rpy="0 0 0"/>
       <geometry>
         <box size="0.266 0.266 0.094"/>
       </geometry>
-    </collision> -->
-    <!-- <inertial>
+    </collision>
+    <inertial>
       <origin xyz="0 0 0" rpy="0 0 0"/>
       <mass value="1.3729096e+00"/>
@@ -71,5 +73,5 @@
                iyy="8.6195418e-03" iyz="-3.5422299e-06"
                izz="1.4612727e-02" />
-    </inertial> -->
+    </inertial>
   </link>
   <joint name="wheel_left_joint" type="continuous">
@@ -92,4 +94,10 @@
         <cylinder length="0.018" radius="0.033"/>
       </geometry>
+      <surface>
+    <contact>
+      <collide_without_contact>false</collide_without_contact>
+      <collide_without_contact_bitmask>${collision_bitmap} | 0x0F</collide_without_contact_bitmask>
+    </contact>
+  </surface>
     </collision>
     <inertial>
@@ -120,4 +128,10 @@
         <cylinder length="0.018" radius="0.033"/>
       </geometry>
+      <surface>
+    <contact>
+      <collide_without_contact>false</collide_without_contact>
+      <collide_without_contact_bitmask>${collision_bitmap} | 0x0F</collide_without_contact_bitmask>
+    </contact>
+  </surface>
     </collision>
     <inertial>
@@ -140,4 +154,10 @@
         <box size="0.030 0.009 0.020"/>
       </geometry>
+      <surface>
+    <contact>
+      <collide_without_contact>false</collide_without_contact>
+      <collide_without_contact_bitmask>${collision_bitmap} | 0x0F</collide_without_contact_bitmask>
+    </contact>
+  </surface>
     </collision>
     <inertial>
@@ -160,4 +180,10 @@
         <box size="0.030 0.009 0.020"/>
       </geometry>
+      <surface>
+    <contact>
+      <collide_without_contact>false</collide_without_contact>
+      <collide_without_contact_bitmask>${collision_bitmap} | 0x0F</collide_without_contact_bitmask>
+    </contact>
+  </surface>
     </collision>
     <inertial>
@@ -189,11 +215,17 @@
       <material name="dark"/>
     </visual>
-    <!-- <collision>
+    <collision>
       <origin xyz="0.015 0 -0.0065" rpy="0 0 0"/>
       <geometry>
         <cylinder length="0.0315" radius="0.055"/>
       </geometry>
-    </collision> -->
-    <!-- <inertial>
+      <surface>
+    <contact>
+      <collide_without_contact>true</collide_without_contact>
+      <collide_without_contact_bitmask>${collision_bitmap}</collide_without_contact_bitmask>
+    </contact>
+  </surface>
+    </collision>
+    <inertial>
       <mass value="0.114" />
       <origin xyz="0 0 0" />
@@ -201,5 +233,5 @@
                iyy="0.001" iyz="0.0"
                izz="0.001" />
-    </inertial> -->
+    </inertial>
   </link>
   <joint name="camera_joint" type="fixed">
@@ -215,12 +247,18 @@
       </geometry>
     </visual>
-    <!-- <collision>
+    <collision>
       <origin xyz="0.003 0.065 0.007" rpy="0 0 0"/>
       <geometry>
         <box size="0.012 0.132 0.020"/>
       </geometry>
-    </collision> -->
+      <surface>
+    <contact>
+      <collide_without_contact>true</collide_without_contact>
+      <collide_without_contact_bitmask>${collision_bitmap}</collide_without_contact_bitmask>
+    </contact>
+  </surface>
+    </collision>
     <!-- This inertial field needs doesn't contain reliable data!! -->
-<!--   <inertial>
+  <inertial>
       <mass value="0.564" />
       <origin xyz="0 0 0" />
@@ -228,5 +266,5 @@
                iyy="0.000498940" iyz="0.0"
                izz="0.003879257" />
-    </inertial>-->
+    </inertial>
   </link>
   <joint name="camera_rgb_joint" type="fixed">
@@ -256,4 +294,4 @@
   </joint>
   <link name="camera_depth_optical_frame"/>
-  <xacro:gazebo_specific frame_prefix="${frame_prefix}" topic_prefix="${topic_prefix}"/>
+  <xacro:gazebo_specific frame_prefix="${frame_prefix}" topic_prefix="${topic_prefix}" collision_bitmap="${collision_bitmap}"/>
 </robot>
